File: Breakout.sch (EAGLE design)
At the start: 178 parts, among them IC1 LM337LZ, IC2 78L05SMD, U1 ADS131E08, U11 TC1014, U12 LTC6655, U2 TLV433, U3 TLV433, U4 TLV433, U5 TLV433, U6 TLV433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

Commit message: Clean PSU
Parts:
- added C84, C86: 100µ, passives-custom:UWT1C6.3X5.4
- added C85, C87: 1µ, resistor:C-EUC0805
- added L1, L2: 180µ, passives-custom:NPIM104P
- added Q1, Q2: 2N3904, transistor-small-signal:2N3904
- added Q3, Q4: 2N3906, transistor-small-signal:2N3906
- added R39, R40: 330, resistor:R-EU_R0603
Connections:
- new net N$6436: C73.2, U$2.OUT
- new net N$6440: L1.2, R39.2
- new net N$6441: C84.+, L1.1, Q1.B
- new net N$6442: Q1.E, Q2.B
- new net N$6443: C86.+, L2.1, Q3.B
- new net N$6446: Q1.C, Q2.C, R39.1
- new net N$6447: C85.1, Q2.E
- new net N$6448: L2.2, R40.2
- new net N$6449: Q3.E, Q4.B
- new net N$6450: Q3.C, Q4.C, R40.1
- new net N$6451: C87.1, Q4.E
- net -5V: no longer C73.2, U$2.OUT
- net GND: now also C84.-, C85.2, C86.-, C87.2
Other:
- moved on the sheet: LED1, LED2, R50, R51
