File: Breakout.sch (EAGLE design)
At the start: 177 parts, among them IC1 LM337LZ, IC2 78L05SMD, U1 ADS131E08, U11 TC1014, U12 LTC6655, U2 TLV433, U3 TLV433, U4 TLV433, U5 TLV433, U6 TLV433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

Commit message: Op-amp Power Routed
Parts:
- added C83: 1µ, resistor:C-EUC0603
Connections:
- new net PAS3: C37.1, JP9.2, R17.2, U4B.+IN
- new net PAS4: C43.1, JP10.2, R21.2, U5B.+IN
- new net PAS5: C49.1, JP15.2, R25.2, U6B.+IN
- new net PAS6: C55.1, JP16.2, R29.2, U7B.+IN
- new net PAS7: C61.1, JP19.2, R33.2, U8B.+IN
- new net PAS8: C67.1, JP20.2, R37.2, U9B.+IN
- net PAS1: no longer C37.1, C49.1, C61.1, JP15.2, JP19.2, JP9.2, R17.2, R25.2, R33.2, U4B.+IN, U6B.+IN, U8B.+IN
- net PAS2: no longer C43.1, C55.1, C67.1, JP10.2, JP16.2, JP20.2, R21.2, R29.2, R37.2, U5B.+IN, U7B.+IN, U9B.+IN
- net VCC: now also C83.1
- net VSS: now also C83.2
Other:
- note added: "Channel 5 Input Stage"
- note added: "Channel 6 Input Stage"
- note added: "Channel 7 Input Stage"
- note added: "Channel 8 Input Stage"

Commit message: Modified Board
Parts:
- removed J1: (no value), SparkFun-Connectors:CONN_023.5MM
- removed JP22: (no value), pinhead:PINHD-1X2
- removed JP4: (no value), conn-custom:PINHD-1X6/90
- removed U$2: LM2664, power-custom:LM2664
- added C84: 0µ1, resistor:C-EUC0603
- added R39, R40, R52, R53: (no value), resistor:R-EU_R0603
- added TP2: VSS, SparkFun-Connectors:TEST-POINT3
- added U10: LM2664, power-custom:LM2664
- added U13: 74AVC9112GTX, clock-custom:74AVC9112GTX
- X1: value X-MHz -> 2.048MHz
Connections:
- net DAISY_IN renamed ADC-DAISY_IN
- removed net ADC_CLK_IN: JP22.2, JP3.10
- new net ADC-DRDY: R40.2, U1.DRDY
- new net ADC-PWDN: R52.2, U1.PWDN
- new net ADC-RST: R1.1, R53.2, U1.RESET
- new net ADC-START: R39.2, U1.START
- new net ADC_CLK_OUT: JP2.4, U13.Y2
- new net N$6436: JP24.2, U13.A
- net +3V3: now also C84.1, R41.1, U13.VCC; no longer R41.2
- net +5V: now also U10.SD, U10.V+; no longer J1.1, U$2.SD, U$2.V+
- net -5V: now also U10.OUT; no longer U$2.OUT
- net ADC_CLK: now also U13.Y1; no longer JP2.4, JP24.2
- net CS: now also JP26.4; no longer JP26.1
- net DRDY: now also JP26.1, R40.1; no longer JP26.4, U1.DRDY
- net EXT-CLK: now also JP24.1, JP3.10; no longer JP22.1, JP24.3
- net EXT-OSC: now also JP24.3; no longer JP24.1
- net GND: now also C84.2, U$4.1, U$4.18, U10.GND, U13.GND, U13.OE; no longer C15.2, C16.2, C17.2, C18.2, C19.2, J1.2, U$2.GND
- net MISO: now also JP26.2; no longer JP26.5
- net MOSI: now also JP26.8; no longer JP26.3
- net N$1: now also R41.2; no longer R41.1
- net N$6434: now also U10.CAP+; no longer U$2.CAP+
- net N$6435: now also U10.CAP-; no longer U$2.CAP-
- net PWDN: now also JP26.7, R52.1; no longer JP26.6, U1.PWDN
- net RST: now also JP26.6, R53.1; no longer JP26.8, R1.1, U1.RESET
- net SCLK: now also JP26.3; no longer JP26.7
- net START: now also JP26.5, R39.1; no longer JP26.2, U1.START
- net VSS: now also C15.2, C16.2, C17.2, C18.2, C19.2, TP2.1
Other:
- note added: "+2V5 Supply Generation"
- note added: "+3V3 Supply Generation"
- note added: "-2V5 Supply Generation"
- note added: "50Ω Term"
- note added: "ADC - CLK"
- note added: "ADC - VREF"
- note added: "Clock Source Selection"
- note added: "Connectors"
- note added: "Daisy Chain Headers"
- note added: "Indicator LEDs"
- note added: "Passive / Active Filter Jumpers"
- note added: "SMA Input"
- note removed: "Passive / Active Switches"
