File: Breakout.brd (EAGLE design)
At the start: 80 x 100 mm, 178 parts, among them IC1 LM337LZ, IC2 78L05SMD, U1 ADS131E08, U11 TC1014, U12 LTC6655, U2 TLV433, U3 TLV433, U4 TLV433, U5 TLV433, U6 TLV433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

Commit message: Modified Board
Parts:
- removed J1: (no value), SparkFun-Connectors:SCREWTERMINAL-3.5MM-2
- removed JP22: (no value), pinhead:1X02
- removed JP4: (no value), conn-custom:1X06/90
- removed U$2: LM2664, power-custom:SOT23-6
- added C84: 0µ1, resistor:C0603
- added R39, R40, R52, R53: (no value), resistor:R0603
- added TP2: VSS, SparkFun-Connectors:PAD.03X.03
- added U10: LM2664, power-custom:SOT23-6
- added U13: 74AVC9112GTX, clock-custom:XFDFN-8
- X1: value X-MHz -> 2.048MHz
- moved JP1 25.6 mm to (76.2, 32.0), turned to 90 degrees
- moved R47 19.9 mm to (33.4, 10.0)
- moved C79 19.4 mm to (44.6, 16.9)
- moved C80 19.3 mm to (48.8, 16.9), turned to 0 degrees
- moved IC2 19.1 mm to (46.9, 13.1)
- moved R46 18.8 mm to (37.6, 10.0)
- moved R49 17.5 mm to (38.6, 13.1)
- moved C73 13.5 mm to (59.4, 15.9), turned to 270 degrees
- moved C78 10.4 mm to (65.9, 16.9)
- moved R41 10.2 mm to (13.1, 7.75), turned to 0 degrees
- moved TP1 10.1 mm to (33.9, 33.1)
- moved R42 9.55 mm to (12.2, 15.5)
- moved IC1 9.38 mm to (65.4, 13.0), turned to 270 degrees
- moved C72 8.68 mm to (56.0, 10.2), turned to 0 degrees
- moved R48 8.38 mm to (45.6, 25.0)
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Connections:
- net DAISY_IN renamed ADC-DAISY_IN
- removed net ADC_CLK_IN: JP22.2, JP3.10
- new net ADC-DRDY: R40.2, U1.47
- new net ADC-PWDN: R52.2, U1.35
- new net ADC-RST: R1.1, R53.2, U1.36
- new net ADC-START: R39.2, U1.38
- new net ADC_CLK_OUT: JP2.4, U13.P$6
- new net N$6436: JP24.2, U13.P$2
- net +3V3: now also C84.1, R41.1, U13.P$1; no longer R41.2
- net +5V: now also U10.4, U10.5; no longer J1.1, U$2.4, U$2.5
- net -5V: now also U10.2; no longer U$2.2
- net ADC_CLK: now also U13.P$5; no longer JP2.4, JP24.2
- net CS: now also JP26.4; no longer JP26.1
- net DRDY: now also JP26.1, R40.1; no longer JP26.4, U1.47
- net EXT-CLK: now also JP24.1, JP3.10; no longer JP22.1, JP24.3
- net EXT-OSC: now also JP24.3; no longer JP24.1
- net GND: now also C84.2, U$4.1, U$4.18, U10.1, U13.P$3, U13.P$4; no longer C15.2, C16.2, C17.2, C18.2, C19.2, J1.2, U$2.1
- net MISO: now also JP26.2; no longer JP26.5
- net MOSI: now also JP26.8; no longer JP26.3
- net N$1: now also R41.2; no longer R41.1
- net N$6434: now also U10.6; no longer U$2.6
- net N$6435: now also U10.3; no longer U$2.3
- net PWDN: now also JP26.7, R52.1; no longer JP26.6, U1.35
- net RST: now also JP26.6, R53.1; no longer JP26.8, R1.1, U1.36
- net SCLK: now also JP26.3; no longer JP26.7
- net START: now also JP26.5, R39.1; no longer JP26.2, U1.38
- net VSS: now also C15.2, C16.2, C17.2, C18.2, C19.2, TP2.P$1
Routing:
- net VSS: track 371.8 -> 285.2 mm, vias 18 -> 14
- net ADC_CLK: track 97.3 -> 22.9 mm
- net +5V: track 109.5 -> 52.3 mm, vias 4 -> 0
- net DRDY: track 83.1 -> 27.2 mm, vias 4 -> 0
- net VCC: track 378.2 -> 326.6 mm, vias 23 -> 19
- net ADC-RST: track 0.00 -> 32.7 mm, vias 0 -> 2
- net RST: track 37.6 -> 10.2 mm
- net PWDN: track 34.8 -> 9.73 mm
- net -5V: track 33.5 -> 11.1 mm
- net ADC_CLK_IN: track 21.4 -> 0.00 mm
- net ADC-MOSI: track 2.57 -> 20.7 mm
- net ADC-PWDN: track 0.00 -> 17.4 mm
- net ADC-CS: track 2.97 -> 20.1 mm
- net ADC-START: track 0.00 -> 17.1 mm
- net ADC-SCLK: track 3.16 -> 16.7 mm
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- removed copper zone on layer 16, net GND
Other:
- outline, holes or cut-outs redrawn
- board text added: "+5V GND"
- board text removed: "+5V"
- board text removed: "2.048 MHz SG5032CAN 50 ppm"
- board text removed: "5V GND"
- board text removed: "MCU Header"
